Commit message: phase 2 of nabled extensions

File: crates/nabled/tests/fixtures/physical_ai/planar2r.urdf (robot description, URDF)
Before this commit: robot planar2r, 1 links, 2 joints
Links:
- added link link1, mass 1.0
- added link link2, mass 1.0
Joints:
- joint j1: axis (none) -> 0 0 1; limit (none) -> lower=-3.14159 upper=3.14159 effort=10 velocity=1; origin xyz=0 0 0 rpy=0 0 0 -> xyz=1 0 0 rpy=0 0 0
- joint j2: axis (none) -> 0 0 1; limit (none) -> lower=-3.14159 upper=3.14159 effort=10 velocity=1
